File: hardware/picflash-board.kicad_pcb (KiCad board)
At the start: 4 copper layers, 72 x 44 mm, 115 parts, among them J1 USB-C, J2 ICSP, J3 SWD, Q1 AO3401A, Q2 2N7002, Q3 2N7002, SW1 BOOTSEL, SW2 RESET, U1 RP2040, U10 SN74LVC1T45DBV, U11 MT3608, U12 TLV75801PDBV, U2 USBLC6-2SC6, U3 AP2112K-3.3, U4 W25Q16JVSSIQ, U5 SN74LVC1T45DBV, U6 SN74LVC1T45DBV, U7 SN74LVC1T45DBV, U8 SN74LVC1T45DBV, U9 SN74LVC1T45DBV, Y1 12MHz

Commit message: firmware v3 pour la carte, références LCSC
Protocole v3 : CAPS, SET_VPP, SET_VDD, MEASURE et nouveaux statuts.
Firmware en deux variantes (feature board par défaut, pico pour le
prototype) : level shifters, MCLR trois états, VPP et VDD cible régulés
en boucle fermée sur l'ADC, tout coupé à la déconnexion. Côté hôte,
session carte (board.rs) : version, capacités, alimentation, mesure,
VPP d'après la puce, extinction en fin de session ; utilisée par le CLI,
picflash-ipecmd et l'interface. Tests contre un modèle du firmware.

Matériel : numéros LCSC pour toute la BOM (catalogue JLCPCB du
15/10/2026), quartz ABM8-272-T3 (charge 10 pF), R10 330 R.

Co-Authored-By: Claude Opus 5.5 <noreply@anthropic.com>
Parts:
- R10: value 1k -> 330
