File: hardware/picflash-board.kicad_sch (KiCad schematic)
At the start: 113 parts, among them J1 USB-C, J2 ICSP, J3 SWD, Q1 AO3401A, Q2 2N7002, Q3 2N7002, SW1 BOOTSEL, SW2 RESET, U1 RP2040, U10 SN74LVC1T45DBV, U11 MT3608, U12 TLV75801PDBV, U2 USBLC6-2SC6, U3 AP2112K-3.3, U4 W25Q16JVSSIQ, U5 SN74LVC1T45DBV, U6 SN74LVC1T45DBV, U7 SN74LVC1T45DBV, U8 SN74LVC1T45DBV, U9 SN74LVC1T45DBV, Y1 12MHz

Commit message: hardware: PCB 4 couches routé et fichiers JLCPCB
Placement par script pcbnew, vias de plan pour chaque pastille GND/+3V3,
routage des signaux par Freerouting (plans internes réservés), plans de
masse externes, export Gerber/BOM/CPL. DRC KiCad : 0 erreur, 0 non
connecté.

Revue globale : R62 15k (VDD cible jusqu'à 4,86 V), C43 en entrée du
MT3608, classe Power 0,4 mm, couches internes déclarées "power" (plus
aucune piste dessus), DIR de U10 tiré au 3V3 via R31. Brochage J2
recoupé avec le PICkit 4. Non testé sur matériel.

Co-Authored-By: Claude Opus 5.5 <noreply@anthropic.com>
Parts:
- added C43: 10u, Capacitor_SMD:C_0805_2012Metric, symbol Device:C
- added R31: 10k, Resistor_SMD:R_0603_1608Metric, symbol Device:R
- R62: value 22k -> 15k
- TP1, TP2, TP3, TP4, TP5: now left out of the parts list
Connections:
- net +3V3: now also R31.1; no longer U10.5 (DIR)
- net +5V: now also C43.1
- net GND: now also C43.2
- new net MCLR_LV_DIR: R31.2, U10.5 (DIR)
Other:
- note added: "VDD cible : TLV75801, 1,5-4,85 V"
- note removed: "VDD cible : TLV75801, 1,5-5 V"
Changed lines of the file:
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@@
     (unit 1)
     (exclude_from_sim no)
-    (in_bom yes)
+    (in_bom no)
     (on_board yes)
     (dnp no)
@@
     (unit 1)
     (exclude_from_sim no)
-    (in_bom yes)
+    (in_bom no)
     (on_board yes)
     (dnp no)
@@
     (unit 1)
     (exclude_from_sim no)
-    (in_bom yes)
+    (in_bom no)
     (on_board yes)
     (dnp no)
@@
     (unit 1)
     (exclude_from_sim no)
-    (in_bom yes)
+    (in_bom no)
     (on_board yes)
     (dnp no)
@@
     (unit 1)
     (exclude_from_sim no)
-    (in_bom yes)
+    (in_bom no)
     (on_board yes)
     (dnp no)
@@
 )
   (label
-    "+3V3"
+    "MCLR_LV_DIR"
     (at 335.28 226.06 180)
     (effects (font (size 1.27 1.27)) (justify right bottom))
@@
 )
   (symbol
+    (lib_id "Device:R")
+    (at 358.14 248.92 0)
+    (unit 1)
+    (exclude_from_sim no)
+    (in_bom yes)
+    (on_board yes)
+    (dnp no)
+    (property
+      "Reference"
+      "R31"
+      (at 360.17 248.92 90)
+      (show_name no)
+      (do_not_autoplace no)
+      (effects (font (size 1.27 1.27))))
+    (property
+      "Value"
+      "10k"
+      (at 358.14 248.92 90)
+      (show_name no)
+      (do_not_autoplace no)
+      (effects (font (size 1.27 1.27))))
+    (property
+      "Footprint"
+      "Resistor_SMD:R_0603_1608Metric"
+      (at 358.14 248.92 0)
+      (effects (font (size 1.27 1.27)) (hide yes)))
+    (property "Datasheet" "" (at 358.14 248.92 0) (effects (font (size 1.27 1.27)) (hide yes)))
+    (pin "1")
+    (pin "2")
+    (instances
+      (project
+        "picflash-board"
+        (path "/e5d87253-6bb0-5339-b794-f0b5a13249f7" (reference "R31") (unit 1)))))
+  (wire
+    (pts (xy 358.14 245.11) (xy 358.14 242.57))
+    (stroke (width 0) (type default))
+)
+  (label
+    "+3V3"
+    (at 358.14 242.57 90)
+    (effects (font (size 1.27 1.27)) (justify left bottom))
+)
+  (wire
+    (pts (xy 358.14 252.73) (xy 358.14 255.27))
+    (stroke (width 0) (type default))
+)
+  (label
+    "MCLR_LV_DIR"
+    (at 358.14 255.27 270)
+    (effects (font (size 1.27 1.27)) (justify right bottom))
+)
+  (symbol
     (lib_id "Device:D_Schottky")
     (at 370.84 248.92 0)
@@
   (no_connect (at 55.88 170.18))
   (symbol
+    (lib_id "Device:C")
+    (at 27.94 170.18 0)
+    (unit 1)
+    (exclude_from_sim no)
+    (in_bom yes)
+    (on_board yes)
+    (dnp no)
+    (property
+      "Reference"
+      "C43"
+      (at 28.58 167.64 0)
+      (show_name no)
+      (do_not_autoplace no)
+      (effects (font (size 1.27 1.27)) (justify left)))
+    (property
+      "Value"
+      "10u"
+      (at 28.58 172.72 0)
+      (show_name no)
+      (do_not_autoplace no)
+      (effects (font (size 1.27 1.27)) (justify left)))
+    (property
+      "Footprint"
+      "Capacitor_SMD:C_0805_2012Metric"
+      (at 27.94 170.18 0)
+      (effects (font (size 1.27 1.27)) (hide yes)))
+    (property "Datasheet" "" (at 27.94 170.18 0) (effects (font (size 1.27 1.27)) (hide yes)))
+    (pin "1")
+    (pin "2")
+    (instances
+      (project
+        "picflash-board"
+        (path "/e5d87253-6bb0-5339-b794-f0b5a13249f7" (reference "C43") (unit 1)))))
+  (wire
+    (pts (xy 27.94 166.37) (xy 27.94 163.83))
+    (stroke (width 0) (type default))
+)
+  (label
+    "+5V"
+    (at 27.94 163.83 90)
+    (effects (font (size 1.27 1.27)) (justify left bottom))
+)
+  (wire
+    (pts (xy 27.94 173.99) (xy 27.94 176.53))
+    (stroke (width 0) (type default))
+)
+  (label
+    "GND"
+    (at 27.94 176.53 270)
+    (effects (font (size 1.27 1.27)) (justify right bottom))
+)
+  (symbol
     (lib_id "Device:L")
     (at 78.74 160.02 0)
@@
     (property
       "Value"
-      "22k"
+      "15k"
       (at 393.7 160.02 90)
       (show_name no)
@@
 )
   (text
-    "VDD cible : TLV75801, 1,5-5 V"
+    "VDD cible : TLV75801, 1,5-4,85 V"
     (exclude_from_sim no)
     (at 322 142 0)

Commit message: firmware v3 pour la carte, références LCSC
Protocole v3 : CAPS, SET_VPP, SET_VDD, MEASURE et nouveaux statuts.
Firmware en deux variantes (feature board par défaut, pico pour le
prototype) : level shifters, MCLR trois états, VPP et VDD cible régulés
en boucle fermée sur l'ADC, tout coupé à la déconnexion. Côté hôte,
session carte (board.rs) : version, capacités, alimentation, mesure,
VPP d'après la puce, extinction en fin de session ; utilisée par le CLI,
picflash-ipecmd et l'interface. Tests contre un modèle du firmware.

Matériel : numéros LCSC pour toute la BOM (catalogue JLCPCB du
15/10/2026), quartz ABM8-272-T3 (charge 10 pF), R10 330 R.

Co-Authored-By: Claude Opus 5.5 <noreply@anthropic.com>
Parts:
- C1, C14, C15, C41, C50, C51, C52: LCSC (none) -> C15849
- C10, C11, C12, C13, C16, C17, C20, C21, C22, C23, C24, C25, C26, C27, C28, C29, C30, C31, C42, C53, C6, C7, C8, C9: LCSC (none) -> C14663
- C2, C43: LCSC (none) -> C15850
- C3: LCSC (none) -> C45783
- C4, C5: LCSC (none) -> C1644
- C40: LCSC (none) -> C12891
- D2: LCSC (none) -> C12624
- D3: LCSC (none) -> C2287
- D4: LCSC (none) -> C2286
- D5: LCSC (none) -> C7502694
- F1: LCSC (none) -> C720075
- J2: LCSC (none) -> C22436149
- J3: LCSC (none) -> C22438100
- L1: LCSC (none) -> C354592
- R1, R2: LCSC (none) -> C23186
- R10: value 1k -> 330; LCSC (none) -> C23138
- R11, R12: LCSC (none) -> C23138
- R20, R22, R24, R26, R28, R52: LCSC (none) -> C22775
- R21, R23, R25, R27, R29, R31, R41, R43, R48, R49, R5, R6, R61, R63, R9: LCSC (none) -> C25804
- R3, R4: LCSC (none) -> C25190
- R30, R44, R46, R50, R51, R64, R65: LCSC (none) -> C25803
- R40: LCSC (none) -> C25811
- R42: LCSC (none) -> C23254
- R45: LCSC (none) -> C25819
- R47: LCSC (none) -> C31850
- R53: LCSC (none) -> C22962
- R60: LCSC (none) -> C23206
- R62: LCSC (none) -> C22809
- R66: LCSC (none) -> C23231
- R7, R8: LCSC (none) -> C21190
- SW1, SW2: LCSC (none) -> C221896
- U10, U5, U6, U7, U8, U9: LCSC (none) -> C7843
- U12: LCSC (none) -> C2877852
- U4: LCSC (none) -> C131025
- Y1: LCSC C9002 -> C20625731
